File: hardware/rules/test/t1-main-board-rules-test.kicad_pcb (KiCad board)
At the start: 8 copper layers, 80 x 122.8 mm, 0 parts

Commit message: DFM and reliability DRC rules: holes, edges, assembly, spacing, routing, battery
Thirty product rules from new desk research
(docs/research/2026-10-pcb-dfm-reliability-rules.md): mounting holes
(PCB-H), board edges and panel tabs (PCB-B), assembly (PCB-D), IPC-2221B
termination spacing (PCB-V), copper necks, teardrops and via counts
(PCB-W), battery and heat placement (PCB-L). Every rule name carries its
RFC 0010 quality level, and the existing rules are retagged. Naming
conventions the rules rely on are in hardware/rules/README.md. The test
board fires every rule once in the FAIL column and nothing in PASS.

Co-Authored-By: Claude Opus 5.5 <noreply@anthropic.com>
Claude-Session: https://claude.ai/code/session_014BJ4LyBAxLcpVCphpLCysj
Parts:
- added C1: test, , F.Cu at (45.5, 159.7)
- added C2: test, , F.Cu at (59.5, 159.7)
- added C3: test, , F.Cu at (40.5, 182.7)
- added C4: test, , F.Cu at (54.5, 182.7)
- added C5: test, , F.Cu at (44.2, 190.6)
- added C6: test, , F.Cu at (58.3, 190.6)
- added FID1: test, , F.Cu at (40.5, 205.6)
- added FID2: test, , F.Cu at (54.5, 205.6)
- added H1: test, , F.Cu at (41.1, 138.0)
- added H10: test, , F.Cu at (55.1, 159.7)
- added H11, U1: test, , F.Cu at (41.1, 164.9)
- added H12, U2: test, , F.Cu at (55.1, 164.9)
- added H2: test, , F.Cu at (55.1, 138.0)
- added H3: test, , F.Cu at (41.1, 143.2)
- added H4: test, , F.Cu at (55.1, 143.2)
- added H5: test, , F.Cu at (41.4, 148.8)
- added H6: test, , F.Cu at (55.4, 148.8)
- added H7: test, , F.Cu at (40.5, 156.1)
- added H8: test, , F.Cu at (54.5, 156.1)
- added H9: test, , F.Cu at (41.1, 159.7)
- added R1: test, , F.Cu at (40.3, 32.5)
- added R10: test, , F.Cu at (56.5, 250.7)
- added R11: test, , F.Cu at (40.3, 271.5)
- added R12: test, , F.Cu at (54.3, 271.5)
- added R13: test, , F.Cu at (56.9, 271.5)
- added R14: test, , F.Cu at (41.5, 276.5)
- added R15: test, , F.Cu at (45.5, 276.5)
- added R16: test, , F.Cu at (55.5, 276.5)
- added R17: test, , F.Cu at (59.5, 276.5)
- added R18: test, , F.Cu at (41.5, 281.0)
- added R19: test, , F.Cu at (45.5, 281.0)
- added R2: test, , F.Cu at (54.3, 32.5)
- added R20: test, , F.Cu at (55.5, 281.0)
- added R21: test, , F.Cu at (59.5, 281.0)
- added R3: test, , F.Cu at (40.3, 41.1)
- added R4: test, , F.Cu at (54.3, 41.1)
- added R5: test, , F.Cu at (43.9, 138.0)
- added R6: test, , F.Cu at (57.9, 138.0)
- added R7: test, , F.Cu at (40.5, 170.2)
- added R8: test, , F.Cu at (54.5, 170.2)
- added R9: test, , F.Cu at (42.5, 250.7)
- added TP1: test, , F.Cu at (40.0, 197.6)
- added TP10: test, , F.Cu at (57.0, 241.7)
- added TP11: test, , F.Cu at (40.5, 250.7)
- added TP12: test, , F.Cu at (54.5, 250.7)
- added TP13: test, , F.Cu at (40.5, 264.5)
- added TP14: test, , F.Cu at (54.5, 264.5)
- added TP2: test, , F.Cu at (54.0, 197.6)
- added TP3: test, , F.Cu at (40.5, 219.4)
- added TP4: test, , F.Cu at (54.5, 219.4)
- added TP5: test, , F.Cu at (40.0, 233.7)
- added TP6: test, , F.Cu at (54.0, 233.7)
- added TP7: test, , F.Cu at (40.5, 241.7)
- added TP8: test, , F.Cu at (43.0, 241.7)
- added TP9: test, , F.Cu at (54.5, 241.7)
- added U3: test, , F.Cu at (41.0, 190.6)
- added U4: test, , F.Cu at (55.0, 190.6)
- added U5: test, , F.Cu at (41.5, 301.5)
- added U6: test, , F.Cu at (55.5, 301.5)
Routing:
- net USB2_90D_1: track 0.00 -> 4.80 mm, vias 0 -> 7
- net N29: track 0.00 -> 4.20 mm
- net N28: track 0.00 -> 4.20 mm
- net USB2_90D_2: track 0.00 -> 4.00 mm, vias 0 -> 6
- net MIPI_100D_1: track 0.00 -> 3.20 mm, vias 0 -> 5
- net N34: track 0.00 -> 3.00 mm
- net N33: track 0.00 -> 3.00 mm
- net N27: track 0.00 -> 3.00 mm
- net N26: track 0.00 -> 3.00 mm
- net N21: track 3.00 -> 0.00 mm
- net N19: track 3.00 -> 0.00 mm
- net N25: track 0.00 -> 2.80 mm
- net N46: track 0.00 -> 2.55 mm
- net N45: track 0.00 -> 2.53 mm
- net MIPI_100D_2: track 0.00 -> 2.40 mm, vias 0 -> 4
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- added copper zone on F.Cu, net N54
- added copper zone on F.Cu, net N55
- added copper zone on F.Cu, net N56
- added copper zone on F.Cu, net N57
Other:
- board size 80 x 122.8 mm -> 80 x 312.3 mm
- board text added: "T1 PCB-A-06 [Q1]: Switch node to analog audio"
- board text added: "T1 PCB-A-07 [Q1]: Foreign track in the analog audio area"
- board text added: "T1 PCB-B-01 [Q1]: Part to board edge"
- board text added: "T1 PCB-B-02 [Q1]: Copper to edge at a break tab"
- board text added: "T1 PCB-B-03 [Q1]: MLCC at a break tab"
- board text added: "T1 PCB-D-01 [Q1]: BGA rework clearance"
- board text added: "T1 PCB-D-02 [Q1]: Fiducial size"
- board text added: "T1 PCB-D-03 [Q1]: Fiducial clear area"
- board text added: "T1 PCB-D-04 [Q2]: Fiducial to board edge"
- board text added: "T1 PCB-D-05 [Q2]: Silkscreen to board edge"
- board text added: "T1 PCB-D-06 [Q2]: Test point size"
- board text added: "T1 PCB-D-07 [Q2]: Test point spacing"
- board text added: "T1 PCB-D-08 [Q2]: Test point to other pads"
- board text added: "T1 PCB-D-09 [Q2]: Test point to board edge"
- board text added: "T1 PCB-D-10 [Q1]: Open via near an SMD pad"
- board text added: "T1 PCB-G-01 [Q1]: Copper clearance"
- board text added: "T1 PCB-G-01 [Q1]: Track width"
- board text added: "T1 PCB-G-02 [Q1]: Copper clearance in the BGA escape"
- board text added: "T1 PCB-G-02 [Q1]: Track width in the BGA escape"
- board text added: "T1 PCB-G-03 [Q1]: Microvia diameter"
- board text added: "T1 PCB-G-04 [Q1]: Mechanical via diameter"
- board text added: "T1 PCB-G-05 [Q1]: Copper to board edge"
- board text added: "T1 PCB-H-01 [Q1]: Part under the screw head"
- board text added: "T1 PCB-H-02 [Q1]: Copper under the screw head"
- board text added: "T1 PCB-H-03 [Q2]: Plated mounting hole on GND"
- board text added: "T1 PCB-H-04 [Q1]: Mounting hole to board edge"
- board text added: "T1 PCB-H-05 [Q1]: MLCC to mounting hole"
- board text added: "T1 PCB-H-06 [Q2]: BGA to mounting hole"
- board text added: "T1 PCB-I-09 [Q1]: Master clock to other nets"
- board text added: "T1 PCB-L-01 [Q0]: Hot part at the battery pocket"
- board text added: "T1 PCB-L-02 [Q0]: Foreign track at the battery connector"
- board text added: "T1 PCB-P-01 [Q0]: Battery path track width (inner)"
- board text added: "T1 PCB-P-01 [Q0]: Battery path track width (outer)"
- board text added: "T1 PCB-P-02 [Q0]: VSYS track width (inner)"
- board text added: "T1 PCB-P-02 [Q0]: VSYS track width (outer)"
- board text added: "T1 PCB-P-03 [Q0]: VBUS input track width (inner)"
- board text added: "T1 PCB-P-03 [Q0]: VBUS input track width (outer)"
- board text added: "T1 PCB-P-04 [Q0]: 5.1 V source track width (inner)"
- board text added: "T1 PCB-P-04 [Q0]: 5.1 V source track width (outer)"
- board text added: "T1 PCB-P-05 [Q0]: HAT 3.3 V track width (inner)"
- board text added: "T1 PCB-P-05 [Q0]: HAT 3.3 V track width (outer)"
- board text added: "T1 PCB-P-06 [Q1]: Amplifier rail track width"
- board text added: "T1 PCB-V-01 [Q1]: Exposed termination spacing"
- board text added: "T1 PCB-V-02 [Q1]: VBUS termination spacing"
- board text added: "T1 PCB-W-01 [Q1]: Copper neck"
- board text added: "T1 PCB-W-01 [Q1]: Copper neck in the BGA escape"
- board text added: "T1 PCB-W-02 [Q2]: Teardrops on vias"
- board text added: "T1 PCB-W-03 [Q2]: Vias per MIPI line"
- board text added: "T1 PCB-W-03 [Q2]: Vias per PCIe line"
- board text added: "T1 PCB-W-03 [Q2]: Vias per USB 2 line"
- board text added: "T1 PCB-W-03 [Q2]: Vias per USB 3 line"
- board text removed: "T1 PCB-A-06: Switch node to analog audio"
- board text removed: "T1 PCB-A-07: Foreign track in the analog audio area"
- board text removed: "T1 PCB-G-01: Copper clearance"
- board text removed: "T1 PCB-G-01: Track width"
- board text removed: "T1 PCB-G-02: Copper clearance in the BGA escape"
- board text removed: "T1 PCB-G-02: Track width in the BGA escape"
- board text removed: "T1 PCB-G-03: Microvia diameter"
- board text removed: "T1 PCB-G-04: Mechanical via diameter"
- board text removed: "T1 PCB-G-05: Copper to board edge"
- board text removed: "T1 PCB-I-09: Master clock to other nets"
- board text removed: "T1 PCB-P-01: Battery path track width (inner)"
- board text removed: "T1 PCB-P-01: Battery path track width (outer)"
- board text removed: "T1 PCB-P-02: VSYS track width (inner)"
- board text removed: "T1 PCB-P-02: VSYS track width (outer)"
- board text removed: "T1 PCB-P-03: VBUS input track width (inner)"
- board text removed: "T1 PCB-P-03: VBUS input track width (outer)"
- board text removed: "T1 PCB-P-04: 5.1 V source track width (inner)"
- board text removed: "T1 PCB-P-04: 5.1 V source track width (outer)"
- board text removed: "T1 PCB-P-05: HAT 3.3 V track width (inner)"
- board text removed: "T1 PCB-P-05: HAT 3.3 V track width (outer)"
- board text removed: "T1 PCB-P-06: Amplifier rail track width"

Commit message: PCB design constraints v0.6: DFM families, industry-wisdom gaps, craft net classes
- Constraints: mounting holes (H), edges and panel (B), assembly (D),
  voltage spacing (V), routing hygiene (W) and battery and heat (L) as
  constraint rows with levels; the industry-wisdom gaps under new IDs
  (mapping appended to the gaps note); PCB-I-09 reworded (no guard traces,
  MCLK branch <= 20 mm from sim/mclk-attenuator); PCB-E-04 merges gap G-25.
- Net classes follow the craft convention: MCLK_50SE, I2S_50SE,
  EMMC_SD_50SE, RF_50SE, DDR_50SE, DDR_100D, PCIE_REFCLK_100D.
- hardware/t1-main-board: rule manifest and composed rules (pcbway-hdi,
  opendap-craft, product rules), craft check configuration (target Q1,
  placeholder mirrored blocks).
- kicad-lib submodule to f03a3cc (opendap-craft).

Co-Authored-By: Claude Opus 5.5 <noreply@anthropic.com>
Claude-Session: https://claude.ai/code/session_014BJ4LyBAxLcpVCphpLCysj
Routing:
- net MCLK_50SE_2: track 0.00 -> 3.00 mm
- net MCLK_50SE_1: track 0.00 -> 3.00 mm
- net MCLK_2: track 3.00 -> 0.00 mm
- net MCLK_1: track 3.00 -> 0.00 mm
Changed lines of the file:
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@@
 		(width 0.2)
 		(layer "F.Cu")
-		(net "MCLK_1")
+		(net "MCLK_50SE_1")
 	)
 	(segment
@@
 		(width 0.2)
 		(layer "F.Cu")
-		(net "MCLK_2")
+		(net "MCLK_50SE_2")
 	)
 	(segment

Commit message: BOM v1.10, power tree v0.4, PCB constraints v0.9: battery through contacts (ADR 0020)
- BOM line 47: Micro-Fit 3.0 -> six KYOCERA AVX 70-9258-001-120-006
  (P+, P+, empty, mid-cell tap, NTC, P-, P-); line 46 pack terminal board
  with recessed hard-gold pads and keying; lines 39, 42, 48, 104 wording;
  line 115 BATP 47 nF; new lines 142 (contact ESD, DNP P+ TVS) and 143
  (cover detect, should); freed 2.5 mm lead allowance noted.
- Power tree §4.7.1: BRD-049 margins through the contacts (33 % at 3.2 A,
  52 % at 5 A on the hotter contact), contact resistance and heat.
- PCB constraints: PCB-L-04 to L-10 merged; DRC rules for L-04, L-05,
  L-08 (warning, UNVERIFIED distance); BAT_SENSE net class; test board
  extended; composition regenerated.
- Feature blocks: blk.charger record updated; blk.cover-detect (#50)
  added to the catalog and the three variant files.

Co-Authored-By: Claude Opus 5.5 <noreply@anthropic.com>
Claude-Session: https://claude.ai/code/session_014BJ4LyBAxLcpVCphpLCysj
Parts:
- added D1: test, , F.Cu at (43.5, 318.8)
- added D2: test, , F.Cu at (54.5, 318.8)
- added R22: test, , F.Cu at (41.5, 310.3)
- added R23: test, , F.Cu at (55.5, 310.3)
Routing:
- net N63: track 0.00 -> 2.00 mm
- net N62: track 0.00 -> 2.00 mm
Other:
- board size 80 x 312.3 mm -> 80 x 324.3 mm
- board text added: "T1 PCB-L-02 [Q0]: Foreign track at the battery contacts"
- board text added: "T1 PCB-L-04 [Q0]: Copper at the empty battery contact position"
- board text added: "T1 PCB-L-05 [Q0]: Foreign pad at the battery contacts"
- board text added: "T1 PCB-L-08 [Q1]: Battery contact ESD away from the contacts"
- board text removed: "T1 PCB-L-02 [Q0]: Foreign track at the battery connector"

Commit message: BOM v1.11, power tree v0.5, constraints v0.10: HAT interface v1.1, faceplate interface v1
Applies hat-standard interface v1.1 and its ADR 0005 to the board:
- One DF40C-100 pair per cable end (87 of 96 usable, corners are metal
  fittings per the DF40 catalog p. 10 note 3); DF40C-50 pair removed.
- 68 pogo pins; HAT ESD TPD4E05U06 x4 + x8, TPD1E10B06 x0 (line out gone).
- New line 144: two TMUXHS4412IRUAR share EXT0-EXT4 between PCIe and
  CSI-2; BRD-042 figures recorded (13 GHz BW, -0.7 dB IL and -23 dB RL at
  2.5 GHz, typical). PCIe TX caps on the SoC side of the switch.
- Limiters against the new fault ceilings, tolerance included: eFuse #A
  1.68 A, eFuse #B 1.16 A; TPS2121 RILM 44.2 -> 45.3 kOhm 0.1 % (3.02 ->
  2.95 A max), charger IINDPM 1.9 A at 5 V.
- Pinout v1 and CSV: A22/B22 -> HAT_EXT_SEL/HAT_EXT_PD, SWD on GPIO2/3,
  sidebands HAT_EXT_SB0-SB2, PHY balls to the switch ports.
- Constraints: HAT_EXT_100D (PCB-I-12), switch placement (PCB-I-13),
  PWR_HAT5V 3.0 A (PCB-P-20), P-04/P-05 at the maximum trips; DRC rules,
  test board regenerated (57/57 PASS), project rules recomposed.

Applies the faceplate interface v1 board changes (t1 e1e18e7):
- FP_3V3 on a TPS22950 (0.22-0.38 A); FP_1V8, MIC_1V8 and FP_VCI on
  TPS22945 (100-200 mA); LDO4 has no stated trip value.
- Backlight TPS61160 (open-LED 25-27 V) with a 22 uH inductor.
- I2C3 pull-ups 2.2 kOhm; identity node in blk.fp-controls; v0 -> v1.

Co-Authored-By: Claude Opus 5.5 <noreply@anthropic.com>
Claude-Session: https://claude.ai/code/session_014BJ4LyBAxLcpVCphpLCysj
Parts:
- removed the H4 at (55.1, 143.2)
- removed the R13 at (56.9, 271.5)
- removed the R17 at (59.5, 276.5)
- added H5: test, , F.Cu at (41.4, 163.7)
- added R14: test, , F.Cu at (41.5, 291.4)
- added R18: test, , F.Cu at (41.5, 295.9)
- moved R17 20.8 mm to (59.5, 291.4)
- moved D1 18.4 mm to (43.5, 337.2)
- moved D2 18.4 mm to (54.5, 337.2)
- moved R22 18.4 mm to (41.5, 328.7)
- moved R23 18.4 mm to (55.5, 328.7)
- moved U5 18.4 mm to (41.5, 319.9)
- moved U6 18.4 mm to (55.5, 319.9)
- moved R13 18.3 mm to (56.9, 286.4)
- moved H4 16.5 mm to (55.1, 158.1)
- moved H8 14.9 mm to (54.5, 171.0)
- moved H6 14.9 mm to (55.4, 163.7)
- moved H7 14.9 mm to (40.5, 171.0)
- moved C1 14.9 mm to (45.5, 174.5)
- moved C2 14.9 mm to (59.5, 174.5)
- moved H10 14.9 mm to (55.1, 174.5)
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- renumbered H5 to H4, R14 to R13, R18 to R17
Connections:
- R13 pad 1: N54 -> N53
- R17 pad 1: N56 -> N55
Routing:
- net HAT_EXT_100D_1: track 0.00 -> 1.60 mm, vias 0 -> 3
- net PWR_HAT5V_4: track 0.00 -> 1.00 mm
- net PWR_HAT5V_3: track 0.00 -> 1.00 mm
- net PWR_HAT5V_2: track 0.00 -> 1.00 mm
- net PWR_HAT5V_1: track 0.00 -> 1.00 mm
- net HAT_EXT_100D_2: track 0.00 -> 0.80 mm, vias 0 -> 2
Other:
- board size 80 x 324.3 mm -> 80 x 342.7 mm
- board text added: "T1 PCB-P-20 [Q0]: HAT 5 V track width (inner)"
- board text added: "T1 PCB-P-20 [Q0]: HAT 5 V track width (outer)"
- board text added: "T1 PCB-W-03 [Q2]: Vias per HAT extension line"

Commit message: Constraints v0.11 and DRC for stackup v1 impedance classes
Applies stackup v1 §7: net classes carry the stackup, outer and inner
width and gap, and their layers; constraints v0.11 updates PCB-S-01 to
S-06, S-11, S-12, adds S-14 (impedance classes on L1, L3, L8, L10 only)
and S-15 (delay matching across layers), the impedance-class exception
to PCB-G-01, widths and gaps in PCB-I-01 to I-09 and I-12, PCB-I-07 as a
microstrip over a cut-out, the RF stack values and RF_CUTOUT (PCB-R-03),
the I-10 pad-void note and the stackup debt in §9.

Product rules for the 10-layer board: per-layer width bands per class
(computed width -5 %/+5 %, floor 0.075 mm), pair-gap minimums as
clearances between the nets of a pair, PCB-S-14 layer rules (including
MCLK inner only and RF outer only), RF line to same-layer ground 0.6 mm,
the RF_CUTOUT cut-out and pour rules, and a PCB-W-01 neck floor for
impedance classes. Width and gap rules are UNVERIFIED warnings until the
DFM review. The test board has ten copper layers; check_drc passes.

Co-Authored-By: Claude Opus 5.5 <noreply@anthropic.com>
Claude-Session: https://claude.ai/code/session_014BJ4LyBAxLcpVCphpLCysj
Parts:
- added R24: test, , F.Cu at (55.5, 300.4)
- added R25: test, , F.Cu at (59.5, 300.4)
- added R26: test, , F.Cu at (41.5, 411.9)
- added R27: test, , F.Cu at (55.5, 411.9)
- moved D1 83.2 mm to (43.5, 420.4)
- moved D2 83.2 mm to (54.5, 420.4)
- moved U5 83.2 mm to (41.5, 403.1)
- moved U6 83.2 mm to (55.5, 403.1)
- moved R23 30.0 mm to (45.5, 300.4)
- moved R22 28.3 mm to (41.5, 300.4)
Connections:
- net N57 renamed DDR_50SE_2
- R18 pad 1: N56 -> DDR_50SE_1
- R19 pad 1: N56 -> DDR_50SE_1
- R22 pad 1: N61 -> N56
- R23 pad 1: BAT_SENSE_1 -> N56
Routing:
- net GND: track 0.00 -> 279.0 mm, vias 0 -> 5
- net USB3_90D_5: track 0.00 -> 3.00 mm
- net USB3_90D_4: track 0.00 -> 3.00 mm
- net USB3_90D_3: track 0.00 -> 3.00 mm
- net USB2_90D_9_P: track 0.00 -> 3.00 mm
- net USB2_90D_9_N: track 0.00 -> 3.00 mm
- net USB2_90D_8_P: track 0.00 -> 3.00 mm
- net USB2_90D_8_N: track 0.00 -> 3.00 mm
- net USB2_90D_7: track 0.00 -> 3.00 mm
- net USB2_90D_6: track 0.00 -> 3.00 mm
- net USB2_90D_5: track 0.00 -> 3.00 mm
- net RF_50SE_7: track 0.00 -> 3.00 mm
- net RF_50SE_6: track 0.00 -> 3.00 mm
- net RF_50SE_5: track 0.00 -> 3.00 mm
- net RF_50SE_4: track 0.00 -> 3.00 mm
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- added copper zone on F.Cu, net DDR_50SE_1
- added copper zone on In1.Cu, net GND
- added copper zone on F.Cu, net N57
Other:
- board size 80 x 342.7 mm -> 80 x 425.9 mm
- copper layers 8 -> 10
- board text added: "T1 PCB-I-01/02 [Q1]: 90 ohm pair width (inner)"
- board text added: "T1 PCB-I-01/02 [Q1]: 90 ohm pair width (outer)"
- board text added: "T1 PCB-I-01/02/03 [Q1]: 85 and 90 ohm pair gap (inner)"
- board text added: "T1 PCB-I-01/02/03 [Q1]: 85 and 90 ohm pair gap (outer)"
- board text added: "T1 PCB-I-03 [Q1]: 85 ohm pair width (inner)"
- board text added: "T1 PCB-I-03 [Q1]: 85 ohm pair width (outer)"
- board text added: "T1 PCB-I-03/04/05/12 [Q1]: 100 ohm pair gap (inner)"
- board text added: "T1 PCB-I-03/04/05/12 [Q1]: 100 ohm pair gap (outer)"
- board text added: "T1 PCB-I-03/04/05/12 [Q1]: 100 ohm pair width (inner)"
- board text added: "T1 PCB-I-03/04/05/12 [Q1]: 100 ohm pair width (outer)"
- board text added: "T1 PCB-I-05/06/08 [Q1]: 50 ohm single-ended width (outer)"
- board text added: "T1 PCB-I-05/06/08/09 [Q1]: 50 ohm single-ended width (inner)"
- board text added: "T1 PCB-I-07 [Q1]: RF line to same-layer ground"
- board text added: "T1 PCB-I-07 [Q1]: RF line width"
- board text added: "T1 PCB-R-03 [Q1]: Copper in the RF ground cut-out"
- board text added: "T1 PCB-R-03 [Q1]: Foreign copper on the RF ground pour"
- board text added: "T1 PCB-S-14 [Q1]: Impedance class on a plane layer"
- board text added: "T1 PCB-S-14 [Q1]: Master clock on an outer layer"
- board text added: "T1 PCB-S-14 [Q1]: RF line on an inner layer"
- board text added: "T1 PCB-W-01 [Q1]: Copper neck on impedance classes"
